Commit message: feat(ros2): integrate 700mm hybrid URDF, ros2_control hardware interface, MoveIt 2 SRDF, and Gazebo Harmonic launch

File: ros2/astari_selah_description/urdf/astari_selah.gazebo.xacro (robot description, xacro)
@@ -1,28 +1,143 @@
 <?xml version="1.0"?>
 <robot xmlns:xacro="http://www.ros.org/wiki/xacro">
-  <!-- Gazebo material visual tags -->
+  <!-- ========================================================================= -->
+  <!-- 1. GAZEBO HARMONIC PHYSICAL PROPERTIES & MATERIALS                        -->
+  <!-- ========================================================================= -->
   <gazebo reference="base_link">
     <material>Gazebo/DarkGrey</material>
+    <mu1>0.8</mu1>
+    <mu2>0.8</mu2>
+    <self_collide>false</self_collide>
   </gazebo>
   <gazebo reference="link1_shoulder_yoke">
     <material>Gazebo/Blue</material>
+    <mu1>0.5</mu1>
+    <mu2>0.5</mu2>
+    <self_collide>false</self_collide>
   </gazebo>
   <gazebo reference="link2_upper_arm">
     <material>Gazebo/DarkGrey</material>
+    <mu1>0.5</mu1>
+    <mu2>0.5</mu2>
+    <self_collide>false</self_collide>
   </gazebo>
   <gazebo reference="link3_forearm">
     <material>Gazebo/Blue</material>
+    <mu1>0.5</mu1>
+    <mu2>0.5</mu2>
+    <self_collide>false</self_collide>
   </gazebo>
   <gazebo reference="link4_wrist">
     <material>Gazebo/DarkGrey</material>
+    <mu1>0.5</mu1>
+    <mu2>0.5</mu2>
+    <self_collide>false</self_collide>
   </gazebo>
   <gazebo reference="gripper_base">
     <material>Gazebo/Blue</material>
+    <mu1>0.8</mu1>
+    <mu2>0.8</mu2>
+    <self_collide>false</self_collide>
   </gazebo>
   <gazebo reference="gripper_left_finger">
     <material>Gazebo/DarkGrey</material>
+    <mu1>1.2</mu1>
+    <mu2>1.2</mu2>
+    <kp>100000.0</kp>
+    <kd>1.0</kd>
+    <self_collide>false</self_collide>
   </gazebo>
   <gazebo reference="gripper_right_finger">
     <material>Gazebo/DarkGrey</material>
+    <mu1>1.2</mu1>
+    <mu2>1.2</mu2>
+    <kp>100000.0</kp>
+    <kd>1.0</kd>
+    <self_collide>false</self_collide>
+  </gazebo>
+  <!-- ========================================================================= -->
+  <!-- 2. ESP32-CAM GAZEBO SIMULATION SENSOR (OV2640, 20° downward tilt)         -->
+  <!-- ========================================================================= -->
+  <gazebo reference="camera_link">
+    <sensor type="camera" name="esp32_cam">
+      <update_rate>30.0</update_rate>
+      <camera name="ov2640">
+        <horizontal_fov>1.15</horizontal_fov> <!-- ~66 deg FOV -->
+        <image>
+          <width>640</width>
+          <height>480</height>
+          <format>R8G8B8</format>
+        </image>
+        <clip>
+          <near>0.05</near>
+          <far>5.0</far>
+        </clip>
+      </camera>
+      <topic>/camera/image_raw</topic>
+    </sensor>
+  </gazebo>
+  <!-- ========================================================================= -->
+  <!-- 3. ROS 2 CONTROL HARDWARE INTERFACE (Mock / Hardware / Gazebo)             -->
+  <!-- ========================================================================= -->
+  <ros2_control name="AstariSelahSystem" type="system">
+    <hardware>
+      <plugin>mock_components/GenericSystem</plugin>
+    </hardware>
+    <joint name="joint1_base_yaw">
+      <command_interface name="position">
+        <param name="min">0.1745</param>
+        <param name="max">2.9671</param>
+      </command_interface>
+      <state_interface name="position">
+        <param name="initial_value">1.5708</param>
+      </state_interface>
+      <state_interface name="velocity"/>
+    </joint>
+    <joint name="joint2_shoulder_pitch">
+      <command_interface name="position">
+        <param name="min">0.0</param>
+        <param name="max">1.5708</param>
+      </command_interface>
+      <state_interface name="position">
+        <param name="initial_value">1.5708</param>
+      </state_interface>
+      <state_interface name="velocity"/>
+    </joint>
+    <joint name="joint3_elbow_pitch">
+      <command_interface name="position">
+        <param name="min">0.0</param>
+        <param name="max">2.0944</param>
+      </command_interface>
+      <state_interface name="position">
+        <param name="initial_value">0.7854</param>
+      </state_interface>
+      <state_interface name="velocity"/>
+    </joint>
+    <joint name="joint4_wrist_pitch">
+      <command_interface name="position">
+        <param name="min">-1.5708</param>
+        <param name="max">1.5708</param>
+      </command_interface>
+      <state_interface name="position">
+        <param name="initial_value">0.0</param>
+      </state_interface>
+      <state_interface name="velocity"/>
+    </joint>
+    <joint name="joint5_gripper_left">
+      <command_interface name="position">
+        <param name="min">0.0</param>
+        <param name="max">0.7854</param>
+      </command_interface>
+      <state_interface name="position">
+        <param name="initial_value">0.0</param>
+      </state_interface>
+      <state_interface name="velocity"/>
+    </joint>
+  </ros2_control>
+  <!-- Gazebo Sim ros2_control plugin -->
+  <gazebo>
+    <plugin filename="gz_ros2_control-system" name="gz_ros2_control::GazeboSimROS2ControlPlugin">
+      <parameters>$(find astari_selah_description)/config/ros2_controllers.yaml</parameters>
+    </plugin>
   </gazebo>
 </robot>
